Commit message: test gmapping

File: PN60/cart_core/robot_model/urdf/golf_cart.urdf (robot description, URDF)
Before this commit: robot cart_core, 4 links, 3 joints
Links:
- added link base_footprint
Joints:
- added joint base2footprint: type fixed, parent base_link, child base_footprint, origin xyz=0.0 0.0 -1.75 rpy=0.0 0.0 0
- joint base2laser_link: origin xyz=0.0 0.0 0.55 rpy=0.0 0.0 0 -> xyz=0.0 0.0 0.37 rpy=0.0 0.0 0
- joint base2velodyne: origin xyz=0.0 0.0 0.55 rpy=0.0 0.0 0 -> xyz=0.0 0.0 0.37 rpy=0.0 0.0 0
- joint realsense2base: origin xyz=0.08 0 0.33 rpy=0 0 0 -> xyz=0.1 0 0.35 rpy=0 0 0
